File: FirstSketch_1.brd (EAGLE design)
At the start: 69.8 x 69.7 mm, 41 parts

Commit message: Modified letter after Friday's class.
Parts:
- added LED16, LED17: (no value), homemade-hardware:CHIP-LED0805
- added R18, R19: 470, homemade-hardware:0805
- moved U$7 28.0 mm to (47.8, 14.3)
- moved R1 27.7 mm to (21.6, 16.9), turned to 180 degrees
- moved C1 24.2 mm to (33.4, 28.1)
- moved R10 19.0 mm to (11.0, 65.0), turned to 0 degrees
- moved LED15 16.0 mm to (43.0, 45.0), turned to 270 degrees
- moved R12 15.3 mm to (28.0, 64.0), turned to 90 degrees
- moved C2 15.0 mm to (32.3, 15.3)
- moved U$2 13.2 mm to (18.5, 10.6)
- moved LED8 13.0 mm to (14.0, 65.0), turned to 270 degrees
- moved R14 12.4 mm to (40.0, 63.0), turned to 0 degrees
- moved R15 12.4 mm to (40.0, 56.0), turned to 270 degrees
- moved U$3 11.4 mm to (33.0, 37.0)
- moved R13 11.3 mm to (35.0, 65.0), turned to 0 degrees
- moved LED9 11.0 mm to (22.0, 65.0), turned to 90 degrees
- moved R17 11.0 mm to (40.0, 45.0), turned to 0 degrees
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Connections:
- net N$1 renamed RESET
- net N$10 renamed A3/D3
- net N$11 renamed SCK
- net N$12 renamed MISO
- net N$2 renamed MOSI
- net N$9 renamed A2/D4
- new net N$2: LED16.A, R18.2
- new net N$9: LED17.A, R19.2
- net LED2TRANSISTOR: now also LED16.C, LED17.C
- net POWER: now also R18.1, R19.1
Routing:
- net POWER: track 249.9 -> 184.0 mm
- net RESET: track 63.0 -> 12.0 mm
- net LED2TRANSISTOR: track 98.1 -> 117.4 mm, vias 3 -> 0
- net GND: track 103.1 -> 91.2 mm, vias 4 -> 0
- net A3/D3: track 9.29 -> 17.7 mm, vias 0 -> 2
- net SCK: track 5.73 -> 9.97 mm
- net MOSI: track 14.8 -> 10.9 mm
- net MISO: track 5.81 -> 9.73 mm
- net N$18: track 5.00 -> 1.80 mm
- net A2/D4: track 17.4 -> 20.2 mm, vias 0 -> 2
- net N$9: track 0.00 -> 2.48 mm
- net N$2: track 0.00 -> 2.16 mm
- net N$4: track 0.00 -> 2.02 mm
- net N$19: track 3.02 -> 1.05 mm
- net N$20: track 3.02 -> 1.12 mm
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Other:
- outline, holes or cut-outs redrawn
